File: PCB/PAF_controller/PAF_controller.kicad_pcb (KiCad board)
At the start: 2 copper layers, 74.9 x 86.4 mm, 26 parts, among them J1 Conn_02x05_Odd_Even, J10 Conn_01x03, J11 Conn_01x03, J12 Conn_01x03, J13 Conn_01x03, J2 Conn_02x10_Odd_Even, J3 Conn_01x06, J4 Conn_01x04, J5 Conn_01x08, J6 Conn_01x03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

Commit message: Gerber for v1.0
Other:
- board text added: "JLINK"
